File: pcb/hack_pad.kicad_sch (KiCad schematic)
At the start: 408 parts, among them J1 Barrel_Jack_Switch, Q1 IRLZ44N, Q2 IRF9540N, Q3 IRF9540N, Q4 IRLZ44N, SW1 SW_Push, SW10 SW_Push, SW100 SW_Push, SW11 SW_Push, SW12 SW_Push, SW13 SW_Push, SW14 SW_Push, SW15 SW_Push, SW16 SW_Push, SW17 SW_Push, SW18 SW_Push, SW19 SW_Push, SW2 SW_Push, SW20 SW_Push, SW21 SW_Push, SW22 SW_Push, SW23 SW_Push, SW24 SW_Push, SW25 SW_Push, SW26 SW_Push, SW27 SW_Push, SW28 SW_Push, SW29 SW_Push, SW3 SW_Push, SW30 SW_Push, SW31 SW_Push, SW32 SW_Push, SW33 SW_Push, SW34 SW_Push, SW35 SW_Push, SW36 SW_Push, SW37 SW_Push, SW38 SW_Push, SW39 SW_Push, SW4 SW_Push, SW40 SW_Push, SW41 SW_Push, SW42 SW_Push, SW43 SW_Push, SW44 SW_Push, SW45 SW_Push, SW46 SW_Push, SW47 SW_Push, SW48 SW_Push, SW49 SW_Push, SW5 SW_Push, SW50 SW_Push, SW51 SW_Push, SW52 SW_Push, SW53 SW_Push, SW54 SW_Push, SW55 SW_Push, SW56 SW_Push, SW57 SW_Push, SW58 SW_Push, SW59 SW_Push, SW6 SW_Push, SW60 SW_Push, SW61 SW_Push, SW62 SW_Push, SW63 SW_Push, SW64 SW_Push, SW65 SW_Push, SW66 SW_Push, SW67 SW_Push, SW68 SW_Push, SW69 SW_Push, SW7 SW_Push, SW70 SW_Push, SW71 SW_Push, SW72 SW_Push, SW73 SW_Push, SW74 SW_Push, SW75 SW_Push, SW76 SW_Push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

Commit message: Done - minus bom
Parts:
- added SW101: SW_Nidec_CAS-120A1, Button_Switch_SMD:Nidec_Copal_CAS-120A, symbol Switch:SW_Nidec_CAS-120A1
- Q1, Q2, Q3, Q4: footprint Package_TO_SOT_THT:TO-220-3_Vertical -> Package_TO_SOT_THT:TO-220-3_Horizontal_TabDown
Connections:
- net VBUS: now also SW101.1 (C)
- net at Brd1.2 (VCC), U1.40 (VBUS): now also SW101.2 (B); no longer D205.1 (K)
- new net: D205.1 (K), SW101.3 (A)
Other:
- moved on the sheet: D205
Changed lines of the file:
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@@
 	)
 	(junction
+		(at 452.12 101.6)
+		(diameter 0)
+		(color 0 0 0 0)
+	)
+	(junction
 		(at 106.68 48.26)
 		(diameter 0)
@@
 	(wire
 		(pts
+			(xy 444.5 101.6) (xy 452.12 101.6)
+		)
+		(stroke
+			(width 0)
+			(type default)
+		)
+	)
+	(wire
+		(pts
 			(xy 157.48 40.64) (xy 157.48 58.42)
 		)
@@
 	(wire
 		(pts
+			(xy 452.12 101.6) (xy 453.39 101.6)
+		)
+		(stroke
+			(width 0)
+			(type default)
+		)
+	)
+	(wire
+		(pts
 			(xy 199.39 255.27) (xy 199.39 271.78)
 		)
@@
 	(wire
 		(pts
+			(xy 452.12 96.52) (xy 452.12 101.6)
+		)
+		(stroke
+			(width 0)
+			(type default)
+		)
+	)
+	(wire
+		(pts
 			(xy 111.76 93.98) (xy 111.76 111.76)
 		)
@@
 	(wire
 		(pts
-			(xy 424.18 99.06) (xy 422.91 99.06)
+			(xy 434.34 99.06) (xy 422.91 99.06)
 		)
 		(stroke
@@
 	)
 	(symbol
+		(lib_id "Switch:SW_Nidec_CAS-120A1")
+		(at 439.42 99.06 0)
+		(unit 1)
+		(exclude_from_sim no)
+		(in_bom yes)
+		(on_board yes)
+		(dnp no)
+		(property "Reference" "SW101"
+			(at 439.42 84.074 0)
+			(effects
+				(font
+					(size 1.27 1.27)
+				)
+			)
+		)
+		(property "Value" "SW_Nidec_CAS-120A1"
+			(at 439.42 86.614 0)
+			(effects
+				(font
+					(size 1.27 1.27)
+				)
+			)
+		)
+		(property "Footprint" "Button_Switch_SMD:Nidec_Copal_CAS-120A"
+			(at 439.42 109.22 0)
+			(effects
+				(font
+					(size 1.27 1.27)
+				)
+				(hide yes)
+			)
+		)
+		(property "Datasheet" "https://www.nidec-components.com/e/catalog/switch/cas.pdf"
+			(at 439.42 106.68 0)
+			(effects
+				(font
+					(size 1.27 1.27)
+				)
+				(hide yes)
+			)
+		)
+		(property "Description" "Switch, single pole double throw"
+			(at 439.42 99.06 0)
+			(effects
+				(font
+					(size 1.27 1.27)
+				)
+				(hide yes)
+			)
+		)
+		(pin "3"
+		)
+		(pin "1"
+		)
+		(pin "2"
+		)
+		(instances
+			(project ""
+				(path "/d4b0ca01-3fca-43e7-acf5-9c62f788d69d"
+					(reference "SW101")
+					(unit 1)
+				)
+			)
+		)
+	)
+	(symbol
 		(lib_id "LED:SK6812MINI")
 		(at 222.25 302.26 0)
@@
 	(symbol
 		(lib_id "Device:D")
-		(at 427.99 99.06 0)
+		(at 448.31 96.52 0)
 		(unit 1)
 		(exclude_from_sim no)
@@
 		(fields_autoplaced yes)
 		(property "Reference" "D205"
-			(at 427.99 92.71 0)
+			(at 448.31 90.17 0)
 			(effects
 				(font
@@
 		)
 		(property "Value" "D"
-			(at 427.99 95.25 0)
+			(at 448.31 92.71 0)
 			(effects
 				(font
@@
 		)
 		(property "Footprint" "Diode_SMD:D_SMA_Handsoldering"
-			(at 427.99 99.06 0)
+			(at 448.31 96.52 0)
 			(effects
 				(font
@@
 		)
 		(property "Datasheet" "~"
-			(at 427.99 99.06 0)
+			(at 448.31 96.52 0)
 			(effects
 				(font
@@
 		)
 		(property "Description" "Diode"
-			(at 427.99 99.06 0)
+			(at 448.31 96.52 0)
 			(effects
 				(font
@@
 		)
 		(property "Sim.Device" "D"
-			(at 427.99 99.06 0)
+			(at 448.31 96.52 0)
 			(effects
 				(font
@@
 		)
 		(property "Sim.Pins" "1=K 2=A"
-			(at 427.99 99.06 0)
+			(at 448.31 96.52 0)
 			(effects
 				(font
@@
 			)
 		)
-		(property "Footprint" "Package_TO_SOT_THT:TO-220-3_Vertical"
+		(property "Footprint" "Package_TO_SOT_THT:TO-220-3_Horizontal_TabDown"
 			(at 559.435 76.2 0)
 			(effects
@@
 			)
 		)
-		(property "Footprint" "Package_TO_SOT_THT:TO-220-3_Vertical"
+		(property "Footprint" "Package_TO_SOT_THT:TO-220-3_Horizontal_TabDown"
 			(at 542.925 66.04 0)
 			(effects
@@
 	(symbol
 		(lib_id "power:VBUS")
-		(at 431.8 99.06 270)
+		(at 453.39 101.6 270)
 		(unit 1)
 		(exclude_from_sim no)
@@
 		(fields_autoplaced yes)
 		(property "Reference" "#PWR0204"
-			(at 427.99 99.06 0)
+			(at 449.58 101.6 0)
 			(effects
 				(font
@@
 		)
 		(property "Value" "VBUS"
-			(at 435.61 99.0599 90)
+			(at 457.2 101.5999 90)
 			(effects
 				(font
@@
 		)
 		(property "Footprint" ""
-			(at 431.8 99.06 0)
+			(at 453.39 101.6 0)
 			(effects
 				(font
@@
 		)
 		(property "Datasheet" ""
-			(at 431.8 99.06 0)
+			(at 453.39 101.6 0)
 			(effects
 				(font
@@
 		)
 		(property "Description" "Power symbol creates a global label with name \"VBUS\""
-			(at 431.8 99.06 0)
+			(at 453.39 101.6 0)
 			(effects
 				(font
@@
 			)
 		)
-		(property "Footprint" "Package_TO_SOT_THT:TO-220-3_Vertical"
+		(property "Footprint" "Package_TO_SOT_THT:TO-220-3_Horizontal_TabDown"
 			(at 555.625 66.04 0)
 			(effects
@@
 			)
 		)
-		(property "Footprint" "Package_TO_SOT_THT:TO-220-3_Vertical"
+		(property "Footprint" "Package_TO_SOT_THT:TO-220-3_Horizontal_TabDown"
 			(at 546.735 76.2 0)
 			(effects

Commit message: asdasd
Parts:
- removed SW101: SW_Nidec_CAS-120A1, Button_Switch_SMD:Nidec_Copal_CAS-120A, symbol Switch:SW_Nidec_CAS-120A1
- added JP1, JP2: SolderJumper_2_Open, Jumper:SolderJumper-2_P1.3mm_Open_Pad1.0x1.5mm, symbol Jumper:SolderJumper_2_Open
- D1, D10, D100, D11, D12, D13, D14, D15, D16, D17, D18, D19, D2, D20, D21, D22, D23, D24, D25, D26, D27, D28, D29, D3, D30, D31, D32, D33, D34, D35, D36, D37, D38, D39, D4, D40, D41, D42, D43, D44, D45, D46, D47, D48, D49, D5, D50, D51, D52, D53, D54, D55, D56, D57, D58, D59, D6, D60, D61, D62, D63, D64, D65, D66, D67, D68, D69, D7, D70, D71, D72, D73, D74, D75, D76, D77, D78, D79, D8, D80, D81, D82, D83, D84, D85, D86, D87, D88, D89, D9, D90, D91, D92, D93, D94, D95, D96, D97, D98, D99: footprint Diode_SMD:D_0805_2012Metric_Pad1.15x1.40mm_HandSolder -> Diode_SMD:D_SOD-123
Connections:
- net VBUS: now also JP2.2 (B)
- net at Brd1.2 (VCC), U1.40 (VBUS): now also JP1.1 (A), JP2.1 (A)
- net at D205.1 (K): now also JP1.2 (B)

Commit message: Level Shifter
Parts:
- removed JP1: SolderJumper_2_Open, Jumper:SolderJumper-2_P1.3mm_Open_Pad1.0x1.5mm, symbol Jumper:SolderJumper_2_Open
- added JP1, JP3: SolderJumper_2_Bridged, Jumper:SolderJumper-2_P1.3mm_Bridged_RoundedPad1.0x1.5mm, symbol Jumper:SolderJumper_2_Bridged
- added JP4: SolderJumper_2_Open, Jumper:SolderJumper-2_P1.3mm_Open_Pad1.0x1.5mm, symbol Jumper:SolderJumper_2_Open
- added Q5: BSS138, Package_TO_SOT_SMD:SOT-23, symbol Transistor_FET:BSS138
- added R1, R2: 10K, Resistor_SMD:R_0201_0603Metric, symbol Device:R_US
Connections:
- net VBUS: now also R2.1
- net LV: now reaches U1.36 (3V3)
- net LV: now also Q5.1 (G), R1.1
- net at Brd1.2 (VCC), JP2.1 (A), U1.40 (VBUS): now also JP1.1 (A)
- net at D205.1 (K): now also JP1.2 (B)
- net LED renamed LED_HV
- net LED_HV: now also JP3.2 (B), JP4.2 (B); no longer U1.29 (GPIO22)
- new net: JP3.1 (A), Q5.3 (D), R2.2
- new net LED_LV: JP4.1 (A), Q5.2 (S), R1.2, U1.29 (GPIO22)

Commit message: Refactor code structure for improved readability and maintainability
Parts:
- removed JP3: SolderJumper_2_Bridged, Jumper:SolderJumper-2_P1.3mm_Bridged_RoundedPad1.0x1.5mm, symbol Jumper:SolderJumper_2_Bridged
- removed JP4: SolderJumper_2_Open, Jumper:SolderJumper-2_P1.3mm_Open_Pad1.0x1.5mm, symbol Jumper:SolderJumper_2_Open
- R1, R2: footprint Resistor_SMD:R_0201_0603Metric -> Resistor_SMD:R_0603_1608Metric_Pad0.98x0.95mm_HandSolder
Connections:
- net LED_HV: now also Q5.3 (D), R2.2
Changed lines of the file:
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@@
 	)
 	(junction
-		(at 506.73 102.87)
-		(diameter 0)
-		(color 0 0 0 0)
-	)
-	(junction
 		(at 167.64 154.94)
 		(diameter 0)
@@
 	(wire
 		(pts
-			(xy 483.87 105.41) (xy 497.84 105.41)
-		)
-		(stroke
-			(width 0)
-			(type default)
-		)
-	)
-	(wire
-		(pts
 			(xy 142.24 76.2) (xy 142.24 93.98)
 		)
@@
 	(wire
 		(pts
-			(xy 506.73 102.87) (xy 506.73 100.33)
-		)
-		(stroke
-			(width 0)
-			(type default)
-		)
-	)
-	(wire
-		(pts
 			(xy 96.52 22.86) (xy 96.52 40.64)
 		)
@@
 	(wire
 		(pts
-			(xy 506.73 100.33) (xy 505.46 100.33)
-		)
-		(stroke
-			(width 0)
-			(type default)
-		)
-	)
-	(wire
-		(pts
 			(xy 121.92 66.04) (xy 137.16 66.04)
 		)
@@
 	(wire
 		(pts
-			(xy 506.73 105.41) (xy 506.73 102.87)
-		)
-		(stroke
-			(width 0)
-			(type default)
-		)
-	)
-	(wire
-		(pts
 			(xy 50.8 147.32) (xy 50.8 165.1)
 		)
@@
 	(wire
 		(pts
-			(xy 483.87 100.33) (xy 483.87 105.41)
-		)
-		(stroke
-			(width 0)
-			(type default)
-		)
-	)
-	(wire
-		(pts
 			(xy 20.32 40.64) (xy 20.32 58.42)
 		)
@@
 	(wire
 		(pts
-			(xy 505.46 105.41) (xy 506.73 105.41)
-		)
-		(stroke
-			(width 0)
-			(type default)
-		)
-	)
-	(wire
-		(pts
 			(xy 121.92 190.5) (xy 137.16 190.5)
 		)
@@
 	(wire
 		(pts
-			(xy 513.08 102.87) (xy 506.73 102.87)
-		)
-		(stroke
-			(width 0)
-			(type default)
-		)
-	)
-	(wire
-		(pts
 			(xy 35.56 76.2) (xy 35.56 93.98)
 		)
@@
 	(global_label "LED_HV"
 		(shape input)
-		(at 513.08 102.87 0)
+		(at 497.84 100.33 0)
 		(fields_autoplaced yes)
 		(effects
@@
 		)
 		(property "Intersheetrefs" "${INTERSHEET_REFS}"
-			(at 522.899 102.87 0)
+			(at 507.659 100.33 0)
 			(effects
 				(font
@@
 	)
 	(symbol
-		(lib_id "Jumper:SolderJumper_2_Bridged")
-		(at 501.65 100.33 0)
-		(unit 1)
-		(exclude_from_sim no)
-		(in_bom no)
-		(on_board yes)
-		(dnp no)
-		(fields_autoplaced yes)
-		(property "Reference" "JP3"
-			(at 501.65 93.98 0)
-			(effects
-				(font
-					(size 1.27 1.27)
-				)
-			)
-		)
-		(property "Value" "SolderJumper_2_Bridged"
-			(at 501.65 96.52 0)
-			(effects
-				(font
-					(size 1.27 1.27)
-				)
-			)
-		)
-		(property "Footprint" "Jumper:SolderJumper-2_P1.3mm_Bridged_RoundedPad1.0x1.5mm"
-			(at 501.65 100.33 0)
-			(effects
-				(font
-					(size 1.27 1.27)
-				)
-				(hide yes)
-			)
-		)
-		(property "Datasheet" "~"
-			(at 501.65 100.33 0)
-			(effects
-				(font
-					(size 1.27 1.27)
-				)
-				(hide yes)
-			)
-		)
-		(property "Description" "Solder Jumper, 2-pole, closed/bridged"
-			(at 501.65 100.33 0)
-			(effects
-				(font
-					(size 1.27 1.27)
-				)
-				(hide yes)
-			)
-		)
-		(pin "2"
-		)
-		(pin "1"
-		)
-		(instances
-			(project "hack_pad"
-				(path "/d4b0ca01-3fca-43e7-acf5-9c62f788d69d"
-					(reference "JP3")
-					(unit 1)
-				)
-			)
-		)
-	)
-	(symbol
 		(lib_id "power:VBUS")
 		(at 279.4 25.4 0)
@@
 			)
 		)
-		(property "Footprint" "Resistor_SMD:R_0201_0603Metric"
+		(property "Footprint" "Resistor_SMD:R_0603_1608Metric_Pad0.98x0.95mm_HandSolder"
 			(at 497.586 94.234 90)
 			(effects
@@
 			)
 		)
-		(property "Footprint" "Resistor_SMD:R_0201_0603Metric"
+		(property "Footprint" "Resistor_SMD:R_0603_1608Metric_Pad0.98x0.95mm_HandSolder"
 			(at 484.886 94.234 90)
 			(effects
@@
 					(unit 1)
 				)
-			)
-		)
-	)
-	(symbol
-		(lib_id "Jumper:SolderJumper_2_Open")
-		(at 501.65 105.41 0)
-		(unit 1)
-		(exclude_from_sim no)
-		(in_bom no)
-		(on_board yes)
-		(dnp no)
-		(fields_autoplaced yes)
-		(property "Reference" "JP4"
-			(at 501.65 99.06 0)
-			(effects
-				(font
-					(size 1.27 1.27)
-				)
-			)
-		)
-		(property "Value" "SolderJumper_2_Open"
-			(at 501.65 101.6 0)
-			(effects
-				(font
-					(size 1.27 1.27)
-				)
-			)
-		)
-		(property "Footprint" "Jumper:SolderJumper-2_P1.3mm_Open_Pad1.0x1.5mm"
-			(at 501.65 105.41 0)
-			(effects
-				(font
-					(size 1.27 1.27)
-				)
-				(hide yes)
-			)
-		)
-		(property "Datasheet" "~"
-			(at 501.65 105.41 0)
-			(effects
-				(font
-					(size 1.27 1.27)
-				)
-				(hide yes)
-			)
-		)
-		(property "Description" "Solder Jumper, 2-pole, open"
-			(at 501.65 105.41 0)
-			(effects
-				(font
-					(size 1.27 1.27)
-				)
-				(hide yes)
-			)
-		)
-		(pin "2"
-		)
-		(pin "1"
-		)
-		(instances
-			(project "hack_pad"
-				(path "/d4b0ca01-3fca-43e7-acf5-9c62f788d69d"
-					(reference "JP4")
-					(unit 1)
-				)
